Commit message: Fix cuda errors (dofs also takes all actor ids)

File: assets/amp/soccerball.urdf (robot description, URDF)
Before this commit: robot urdf_robot, 1 links, 0 joints
Links:
- link baseLink: geometry collision mesh filename=meshes/soccerball.obj scale=0.22 0.22 0.22; visual mesh filename=meshes/soccerball.obj scale=0.22 0.22 0.22

Commit message: Update asset loading for any asset and any number of instances

File: assets/amp/soccerball.urdf (robot description, URDF)
Before this commit: robot urdf_robot, 1 links, 0 joints
Links:
- link baseLink: mass 10.0 -> 0.45; geometry collision sphere radius=0.11; visual mesh filename=meshes/soccerball.obj scale=0.22 0.22 0.22
